File: CyrWheel_PCB/LEDCyrWheel.sch (EAGLE design)
At the start: 15 parts

Commit message: PCB design work
Parts:
- removed JP4_LED_STRIP_1, JP5_LED_STRIP_2: M01SMDNS, SparkFun:M01SMDNS
- removed U$4: ADAFRUIT_CC3000_WIFI, LEDCyrWheel:ADAFRUIT_CC3000_WIFI
- added IC1: 74LS125N, adafruit:74LS125N
- added LED_CLK, LED_DATA: M01SMDNS, SparkFun:M01SMDNS
- added U$7: ADAFRUIT_BLE_FRIEND_SPI, LEDCyrWheel:ADAFRUIT_BLE_FRIEND_SPI
Connections:
- removed net N$3: U$1.15/A1, U$1.16/A2
- removed net N$4: U$1.12, U$2.MISO, U$4.MISO
- removed net N$5: U$1.13, U$2.SCLK, U$4.CLK
- removed net WIFI_CS: U$1.7, U$4.CS
- removed net WIFI_IRQ: U$1.5, U$4.IRQ
- removed net WIFI_VBEN: U$1.6, U$4.VBEN
- new net BT_CS: U$1.6, U$7.CS
- new net BT_IRQ: U$1.5, U$7.IRQ
- new net BT_RESET: U$1.4, U$7.RST
- new net LED_CLK: IC1B.I, U$1.14/A0
- new net LED_DATA: IC1A.I, U$1.7
- new net MISO: U$1.12, U$2.MISO, U$7.MISO
- new net MOSI: U$1.11, U$2.MOSI, U$7.MOSI
- new net SCK: U$1.13, U$2.SCLK, U$7.SCK
- net GND: now also IC1A.OE, IC1B.OE, IC1P.GND, U$7.GND; no longer U$4.GND
- net N$2: now also IC1B.O, LED_CLK.1; no longer U$1.11, U$2.MOSI, U$4.MOSI
- net N_PIN_2_LED_STRIP: now also IC1A.O, LED_DATA.1; no longer JP4_LED_STRIP_1.1, JP5_LED_STRIP_2.1, U$1.2
- net VIN: now also IC1P.VCC, U$7.VIN; no longer U$4.VIN
Other:
- note added: "This is the 74AHCT125 for 3.3v -> 5v signals"
- note removed: "pin 15 and 16 should be connected together for the Octo library"

Commit message: PCB fixes
Connections:
- net N$6 renamed SDA
- net N$7 renamed SCL
Changed lines of the file:
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@@
 </segment>
 </net>
-<net name="N$6" class="0">
+<net name="SDA" class="0">
 <segment>
 <pinref part="R3" gate="G$1" pin="2"/>
@@
 </segment>
 </net>
-<net name="N$7" class="0">
+<net name="SCL" class="0">
 <segment>
 <pinref part="R4" gate="G$1" pin="2"/>
